Commit message: [ADD]The system is configured to allow control of a person's posture using a GUI.

File: models/human_gazebo_raised_hand/humanSubjectWithMesh.urdf (robot description, URDF)
Before this commit: robot HumanModel, 93 links, 92 joints
Links:
- link Head: geometry collision sphere radius=0.1105; visual mesh filename=package://gz_human_sim/models/human_gazebo_raised_hand/mesh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 scale=1.03030303 1.03030303 1.03030303
- link LeftFoot: geometry collision box size=0.2584 0.0935 0.0663; visual mesh filename=package://gz_human_sim/models/human_gazebo_raised_hand/mesh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 scale=1.03030303 1.03030303 1.03030303
- link LeftForeArm: geometry collision cylinder length=0.24819999999999998 radius=0.0275; visual mesh filename=package://gz_human_sim/models/human_gazebo_raised_hand/mesh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 scale=0.61111111 0.61111111 1.03030303
- link LeftHand: geometry collision box size=0.072 0.1836 0.025; visual mesh filename=package://gz_human_sim/models/human_gazebo_raised_hand/mesh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 scale=0.9 1.03030303 0.55555556
- link LeftLowerLeg: geometry collision cylinder length=0.41819999999999996 radius=0.045; visual mesh filename=package://gz_human_sim/models/human_gazebo_raised_hand/mesh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 scale=0.7826087 0.7826087 1.03030303
- link LeftShoulder: geometry collision cylinder length=0.14676666666666668 radius=0.029; visual mesh filename=package://gz_human_sim/models/human_gazebo_raised_hand/mesh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 scale=0.64444444 0.64444444 1.03030303
- link LeftToe: geometry collision box size=0.002584 0.0935 0.0663; visual mesh filename=package://gz_human_sim/models/human_gazebo_raised_hand/mesh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 scale=1.03030303 1.03030303 1.03030303
- link LeftUpperArm: geometry collision cylinder length=0.3162 radius=0.029; visual mesh filename=package://gz_human_sim/models/human_gazebo_raised_hand/mesh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 scale=0.64444444 0.64444444 1.03030303
- link LeftUpperLeg: geometry collision cylinder length=0.4165 radius=0.0625; visual mesh filename=package://gz_human_sim/models/human_gazebo_raised_hand/mesh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 scale=0.83333333 0.83333333 1.03030303
- link LowerTrunk: geometry collision box size=0.175 0.2958 0.17; visual mesh filename=package://gz_human_sim/models/human_gazebo_raised_hand/mesh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 scale=0.58333333 1.03030303 1.03030303
- link Neck: geometry collision cylinder length=0.08839999999999999 radius=0.0475; visual mesh filename=package://gz_human_sim/models/human_gazebo_raised_hand/mesh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 scale=0.73076923 0.73076923 1.03030303
- link Pelvis: geometry collision box size=0.175 0.3247 0.1326; visual mesh filename=package://gz_human_sim/models/human_gazebo_raised_hand/mesh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 scale=0.58333333 1.03030303 1.03030303
- link RightFoot: geometry collision box size=0.2584 0.0935 0.0663; visual mesh filename=package://gz_human_sim/models/human_gazebo_raised_hand/mesh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 scale=1.03030303 1.03030303 1.03030303
- link RightForeArm: geometry collision cylinder length=0.24819999999999998 radius=0.0275; visual mesh filename=package://gz_human_sim/models/human_gazebo_raised_hand/mesh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 scale=0.61111111 0.61111111 1.03030303
- link RightHand: geometry collision box size=0.072 0.1836 0.025; visual mesh filename=package://gz_human_sim/models/human_gazebo_raised_hand/mesh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 scale=0.9 1.03030303 0.55555556
- link RightLowerLeg: geometry collision cylinder length=0.41819999999999996 radius=0.045; visual mesh filename=package://gz_human_sim/models/human_gazebo_raised_hand/mesh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 scale=0.7826087 0.7826087 1.03030303
- link RightShoulder: geometry collision cylinder length=0.14676666666666668 radius=0.029; visual mesh filename=package://gz_human_sim/models/human_gazebo_raised_hand/mesh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 scale=0.64444444 0.64444444 1.03030303
- link RightToe: geometry collision box size=0.002584 0.0935 0.0663; visual mesh filename=package://gz_human_sim/models/human_gazebo_raised_hand/mesh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 scale=1.03030303 1.03030303 1.03030303
- link RightUpperArm: geometry collision cylinder length=0.3162 radius=0.029; visual mesh filename=package://gz_human_sim/models/human_gazebo_raised_hand/mesh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 scale=0.64444444 0.64444444 1.03030303
- link RightUpperLeg: geometry collision cylinder length=0.4165 radius=0.0625; visual mesh filename=package://gz_human_sim/models/human_gazebo_raised_hand/mesh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 scale=0.83333333 0.83333333 1.03030303
- link UpperTrunk: geometry collision box size=0.175 0.14676667 0.187; visual mesh filename=package://gz_human_sim/models/human_gazebo_raised_hand/mesh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 scale=0.58333333 1.03030303 1.03030303
